File: Hardware/zero star/untitled.kicad_sch (KiCad schematic)
At the start: 47 parts, among them Q1 SS8050, U5 SPL06-001, U6 MPU-6050, U7 QMC5883L, U8 W25Q128JVE, U9 AT7456E, Y2 27Mhz

Commit message: HW v2.5.7: SPI CS pin swap, PCB layout v1, CubeMX update
Parts:
- removed D10, D11, D6: LED_0603, PCM_fab:LED_0603, symbol PCM_fab:LED_0603
- removed R22, R28, R29: 1kΩ, PCM_fab:R_0603, symbol PCM_fab:R_0603
- U6: footprint Sensor_Motion:InvenSense_QFN-24_4x4mm_P0.5mm -> Package_DFN_QFN:QFN-24-1EP_4x4mm_P0.5mm_EP2.6x2.6mm_ThermalVias
Connections:
- net LED_LOG is gone; now on net LED_MODE: R26.2
- net +3.3V: no longer C28.1, C29.1, U5.2 (CSB), U5.6 (VDDIO), U5.8 (VDD)
- net +3.3VA: now also C28.1, C29.1, U5.2 (CSB), U5.6 (VDDIO), U5.8 (VDD)
- net GND: now also U6.25 (GND); no longer U6.18 (GND)
- net LED_GPS: now also R21.2
- net LED_MODE: no longer R2.2
- net LED_SYS: now also R27.2; no longer R21.2
- net LED_VTX: now also R2.2; no longer R27.2
